File: SolarClapboard.kicad_pcb (KiCad board)
At the start: 2 copper layers, 105 parts, among them J1 TEST_2P, J10 TEST_2P, J11 TEST_2P, J12 TEST_2P, J13 TEST_2P, J14 TEST_2P, J15 TEST_2P, J16 TEST_2P, J17 TEST_2P, J18 TEST_2P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

Commit message: Add files via upload
Ready for layout. Fixed test point hole size.
Parts:
- removed G***: LOGO, KNEK-TEK_logo:KNEK-TEK_logo_11mm
- removed REF***: OSHW-Logo_5.7x6mm_SilkScreen, Symbols:OSHW-Logo_5.7x6mm_SilkScreen
- removed TP7, TP8: TEST_1P, CustomFootprints:TestPointHole
- moved J6 141.0 mm to (66.4, 49.3)
- moved J7 139.2 mm to (70.2, 38.6)
- moved J3 137.1 mm to (81.7, 39.1)
- moved J5 136.2 mm to (57.9, 49.8)
- moved J8 132.3 mm to (62.0, 58.8)
- moved TP2 126.5 mm to (80.1, 50.5)
- moved J4 117.5 mm to (95.6, 41.1)
- moved TP1 112.1 mm to (86.7, 50.5)
- moved TP3 100.7 mm to (92.7, 50.0)
- moved TP10 61.1 mm to (116.3, 119.5)
- moved R6 57.4 mm to (112.0, 112.1)
- moved R5 44.8 mm to (122.6, 111.6)
- moved TP9 27.7 mm to (123.6, 119.1)
- moved U2 22.3 mm to (110.6, 37.4)
- moved TP4 20.8 mm to (105.5, 128.0)
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Other:
- rule pad_to_mask_clearance: 0.2 -> 0.1

Commit message: Add files via upload
Layout in progress. Board is <5" x <3"
Parts:
- added Q2: AO3418, TO_SOT_Packages_SMD:SOT-23, F.Cu at (111.4, 85.5)
- added REF**: MountingHole_3.2mm_M3, Mounting_Holes:MountingHole_3.2mm_M3, F.Cu at (201.8, 126.2)
- added REF**: MountingHole_3.2mm_M3, Mounting_Holes:MountingHole_3.2mm_M3, F.Cu at (147.3, 125.9)
- added REF**: MountingHole_3.2mm_M3, Mounting_Holes:MountingHole_3.2mm_M3, F.Cu at (83.7, 126.0)
- added REF**: MountingHole_3.2mm_M3, Mounting_Holes:MountingHole_3.2mm_M3, F.Cu at (201.8, 60.0)
- added REF**: MountingHole_3.2mm_M3, Mounting_Holes:MountingHole_3.2mm_M3, F.Cu at (147.3, 60.0)
- added REF**: MountingHole_3.2mm_M3, Mounting_Holes:MountingHole_3.2mm_M3, F.Cu at (83.8, 60.0)
- added TP34: TEST_1P, CustomFootprints:TestPointHole, F.Cu at (111.4, 106.8)
- added TP35: TEST_1P, CustomFootprints:TestPointHole, F.Cu at (136.1, 106.9)
- added TP36: TEST_1P, CustomFootprints:TestPointHole, F.Cu at (136.1, 109.5)
- added TP37: TEST_1P, CustomFootprints:TestPointHole, F.Cu at (112.5, 89.8)
- added TP38: TEST_1P, CustomFootprints:TestPointHole, F.Cu at (111.4, 96.6)
- added TP39: TEST_1P, CustomFootprints:TestPointHole, F.Cu at (111.4, 99.1)
- added TP40: TEST_1P, CustomFootprints:TestPointHole, F.Cu at (136.1, 101.9)
- added TP41: TEST_1P, CustomFootprints:TestPointHole, F.Cu at (111.4, 109.4)
- added TP42: TEST_1P, CustomFootprints:TestPointHole, F.Cu at (111.4, 111.9)
- added TP43: TEST_1P, CustomFootprints:TestPointHole, F.Cu at (111.4, 117.0)
- added TP44: TEST_1P, CustomFootprints:TestPointHole, F.Cu at (111.4, 119.6)
- added TP45: TEST_1P, CustomFootprints:TestPointHole, F.Cu at (111.4, 122.2)
- added TP46: TEST_1P, CustomFootprints:TestPointHole, F.Cu at (111.4, 127.3)
- added TP7: TEST_1P, CustomFootprints:TestPointHole, F.Cu at (111.4, 101.7)
- added TP8: TEST_1P, CustomFootprints:TestPointHole, F.Cu at (111.4, 104.2)
- C12, C13, C14, C15, C16, C17, C18, C19, C20, C21, D3, D4, D5, L1, Q1, R10: moved to B.Cu
- R7: value 1M -> 10k
- R9: value 188k -> 10.3k
- TP27: value TEST_1P -> GND
- moved TP16 130.2 mm to (202.8, 85.5)
- moved TP18 118.8 mm to (202.8, 92.9)
- moved TP19 116.1 mm to (202.8, 96.6)
- moved TP24 110.7 mm to (202.8, 100.3)
- moved TP17 106.4 mm to (202.8, 89.2)
- moved C21 101.9 mm to (173.7, 126.0), turned to 270 degrees
- moved J1 100.8 mm to (103.9, 64.8), turned to 90 degrees
- moved J17 99.7 mm to (110.1, 114.5)
- moved TP32 98.5 mm to (202.8, 118.7)
- moved R9 96.0 mm to (117.9, 84.6), turned to 180 degrees
- moved TP31 94.7 mm to (202.8, 115.0)
- moved TP15 92.6 mm to (202.8, 81.8)
- moved TP28 91.7 mm to (202.8, 104.0)
- moved J9 89.5 mm to (107.6, 97.1), turned to 270 degrees
- moved J12 87.0 mm to (110.1, 80.9)
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Connections:
- C8 pad 2: GND -> Net-(C8-Pad2)
- J1 pad 1: +3V3 -> VCC
- J12 pad 1: +3V3 -> VCC
- J19 pad 1: (no net) -> Net-(J19-Pad1)
- J19 pad 11: (no net) -> /Epaper_adapter_sheet/TSCL
- J19 pad 12: (no net) -> /Epaper_adapter_sheet/TSDA
- J19 pad 2: (no net) -> Net-(J19-Pad2)
- J19 pad 3: (no net) -> Net-(J19-Pad3)
- J19 pad 30: (no net) -> Net-(J19-Pad30)
- J19 pad 31: (no net) -> Net-(J19-Pad31)
- J19 pad 32: (no net) -> Net-(J19-Pad32)
- J19 pad 33: (no net) -> Net-(J19-Pad33)
- J19 pad 34: (no net) -> Net-(J19-Pad34)
- J19 pad 4: (no net) -> Net-(J19-Pad4)
- J19 pad 5: (no net) -> Net-(J19-Pad5)
- J19 pad 6: (no net) -> Net-(J19-Pad6)
- R9 pad 2: GND -> Net-(C8-Pad2)
- SC1 pad 1: +3V3 -> VCC
- U2 pad 1: (no net) -> Net-(U2-Pad1)
- U2 pad 10: (no net) -> Net-(U2-Pad10)
- U2 pad 12: (no net) -> Net-(U2-Pad12)
- U2 pad 5: (no net) -> Net-(U2-Pad5)
- U2 pad 8: (no net) -> Net-(U2-Pad8)
- U4 pad 5: (no net) -> Net-(U4-Pad5)
- U4 pad 6: (no net) -> Net-(U4-Pad6)
- U4 pad 7: (no net) -> Net-(U4-Pad7)
- U5 pad 0: (no net) -> Net-(TP38-Pad1)
- U5 pad 1: (no net) -> Net-(TP39-Pad1)
- U5 pad 10: (no net) -> Net-(TP45-Pad1)
- U5 pad 12: (no net) -> Net-(TP46-Pad1)
- U5 pad 2: (no net) -> Net-(TP7-Pad1)
- U5 pad 20: (no net) -> Net-(TP36-Pad1)
- U5 pad 21: (no net) -> Net-(TP35-Pad1)
- U5 pad 23: (no net) -> Net-(TP40-Pad1)
- U5 pad 3: (no net) -> Net-(TP8-Pad1)
- U5 pad 4: (no net) -> Net-(TP34-Pad1)
- U5 pad 5: (no net) -> Net-(TP41-Pad1)
- U5 pad 6: (no net) -> Net-(TP42-Pad1)
- U5 pad 8: (no net) -> Net-(TP43-Pad1)
- U5 pad 9: (no net) -> Net-(TP44-Pad1)
- U5 pad AGND: (no net) -> Net-(U5-PadAGND)
- U5 pad Vin: (no net) -> Net-(U5-PadVin)
Routing:
- net +3V3: track 0.00 -> 62.2 mm
- net Net-(C3-Pad1): track 0.00 -> 41.5 mm
- net /SDA: track 0.00 -> 30.4 mm
- net /PV_ADC: track 0.00 -> 28.2 mm
- net /SCL: track 0.00 -> 26.0 mm
- net Net-(J3-Pad1): track 0.00 -> 25.2 mm, vias 0 -> 1
- net /VBat: track 0.00 -> 23.8 mm, vias 0 -> 1
- net Net-(C6-Pad1): track 0.00 -> 22.0 mm
- net Net-(R2-Pad2): track 0.00 -> 21.2 mm
- net /PROG3: track 0.00 -> 19.5 mm
- net VCC: track 0.00 -> 18.7 mm
- net /PROG1: track 0.00 -> 17.8 mm
- net Net-(J8-Pad2): track 0.00 -> 15.5 mm, vias 0 -> 1
- net Net-(TH1-Pad1): track 0.00 -> 13.3 mm, vias 0 -> 1
- net Net-(BT1-Pad1): track 0.00 -> 13.2 mm
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Other:
- board outline added: 125.9 x 74.2 mm
- net class Default: clearance 0.2 -> 0.1778; trace_width 0.25 -> 0.254
- net class PWR added: clearance 0.1778, trace_width 0.508, via_dia 0.6, via_drill 0.4
- rule trace_clearance: 0.2 -> 0.1778
- board text added: "Autumn 2017"
- board text removed: "October - November 2017"
